Commit message: added end effector support

File: models/ur5e/urdf_ros2/ur5e.ros2_control.xacro (robot description, xacro)
@@ -19,124 +19,9 @@
         </xacro:if>
       </hardware>
-      <!-- <joint name="${tf_prefix}shoulder_pan_joint">
-        <xacro:if value="${ros2_control_hardware_type == 'mujoco'}">
-          <param name="position_kp">3000</param>
-          <param name="position_ki">1</param>
-          <param name="position_kd">100</param>
-          <param name="position_i_max">10000</param>
-          <command_interface name="position_pid" />
-        </xacro:if>
-        <xacro:unless value="${ros2_control_hardware_type == 'mujoco'}">
-          <command_interface name="velocity" />
-        </xacro:unless>
-        <state_interface name="position">
-          <param name="initial_value">${initial_positions['shoulder_pan_joint']}</param>
-        </state_interface>
-        <state_interface name="velocity">
-          <param name="initial_value">0.0</param>
-        </state_interface>
-      </joint>
-      <joint name="${tf_prefix}shoulder_lift_joint">
-        <xacro:if value="${ros2_control_hardware_type == 'mujoco'}">
-          <param name="position_kp">3000</param>
-          <param name="position_ki">1</param>
-          <param name="position_kd">100</param>
-          <param name="position_i_max">10000</param>
-          <command_interface name="position_pid" />
-        </xacro:if>
-        <xacro:unless value="${ros2_control_hardware_type == 'mujoco'}">
-          <command_interface name="velocity" />
-        </xacro:unless>
-        <state_interface name="position">
-          <param name="initial_value">${initial_positions['shoulder_lift_joint']}</param>
-        </state_interface>
-        <state_interface name="velocity">
-          <param name="initial_value">0.0</param>
-        </state_interface>
-      </joint>
-      <joint name="${tf_prefix}elbow_joint">
-        <xacro:if value="${ros2_control_hardware_type == 'mujoco'}">
-          <param name="position_kp">3000</param>
-          <param name="position_ki">1</param>
-          <param name="position_kd">100</param>
-          <param name="position_i_max">10000</param>
-          <command_interface name="position_pid" />
-        </xacro:if>
-        <xacro:unless value="${ros2_control_hardware_type == 'mujoco'}">
-          <command_interface name="velocity" />
-        </xacro:unless>
-        <state_interface name="position">
-          <param name="initial_value">${initial_positions['elbow_joint']}</param>
-        </state_interface>
-        <state_interface name="velocity">
-          <param name="initial_value">0.0</param>
-        </state_interface>
-      </joint>
-      <joint name="${tf_prefix}wrist_1_joint">
-        <xacro:if value="${ros2_control_hardware_type == 'mujoco'}">
-          <param name="position_kp">3000</param>
-          <param name="position_ki">1</param>
-          <param name="position_kd">100</param>
-          <param name="position_i_max">10000</param>
-          <command_interface name="position_pid" />
-        </xacro:if>
-        <xacro:unless value="${ros2_control_hardware_type == 'mujoco'}">
-          <command_interface name="velocity" />
-        </xacro:unless>
-        <state_interface name="position">
-          <param name="initial_value">${initial_positions['wrist_1_joint']}</param>
-        </state_interface>
-        <state_interface name="velocity">
-          <param name="initial_value">0.0</param>
-        </state_interface>
-      </joint>
-      <joint name="${tf_prefix}wrist_2_joint">
-        <xacro:if value="${ros2_control_hardware_type == 'mujoco'}">
-          <param name="position_kp">3000</param>
-          <param name="position_ki">1</param>
-          <param name="position_kd">100</param>
-          <param name="position_i_max">10000</param>
-          <command_interface name="position_pid" />
-        </xacro:if>
-        <xacro:unless value="${ros2_control_hardware_type == 'mujoco'}">
-          <command_interface name="velocity" />
-        </xacro:unless>
-        <state_interface name="position">
-          <param name="initial_value">${initial_positions['wrist_2_joint']}</param>
-        </state_interface>
-        <state_interface name="velocity">
-          <param name="initial_value">0.0</param>
-        </state_interface>
-      </joint>
-      <joint name="${tf_prefix}wrist_3_joint">
-        <xacro:if value="${ros2_control_hardware_type == 'mujoco'}">
-          <param name="position_kp">3000</param>
-          <param name="position_ki">1</param>
-          <param name="position_kd">100</param>
-          <param name="position_i_max">10000</param>
-          <command_interface name="position_pid" />
-        </xacro:if>
-        <xacro:unless value="${ros2_control_hardware_type == 'mujoco'}">
-          <command_interface name="velocity" />
-        </xacro:unless>
-        <state_interface name="position">
-          <param name="initial_value">${initial_positions['wrist_3_joint']}</param>
-        </state_interface>
-        <state_interface name="velocity">
-          <param name="initial_value">0.0</param>
-        </state_interface>
-      </joint> -->
       <xacro:macro name="configure_joint" params="joint_name initial_positions joint_name_wo_prefix">
         <joint name="${joint_name}">
           <xacro:if value="${ros2_control_hardware_type == 'mujoco'}">
-            <param name="position_kp">3000</param>
-            <param name="position_ki">0</param>
-            <param name="position_kd">5</param>
-            <param name="position_i_max">10000</param>
             <command_interface name="position" />
           </xacro:if>
-          <xacro:unless value="${ros2_control_hardware_type == 'mujoco'}">
-            <command_interface name="velocity" />
-          </xacro:unless>
           <state_interface name="position">
             <param name="initial_value">${initial_positions[joint_name_wo_prefix]}</param>
@@ -145,13 +30,22 @@
             <!-- <param name="initial_value">0.0</param> -->
           </state_interface>
-          <state_interface name="effort"/>
+          <state_interface name="effort" />
         </joint>
       </xacro:macro>
-      <xacro:configure_joint joint_name="${tf_prefix}shoulder_pan_joint"  initial_positions="${initial_positions}" joint_name_wo_prefix="shoulder_pan_joint"/>
-      <xacro:configure_joint joint_name="${tf_prefix}shoulder_lift_joint" initial_positions="${initial_positions}" joint_name_wo_prefix="shoulder_lift_joint"/>
-      <xacro:configure_joint joint_name="${tf_prefix}elbow_joint"        initial_positions="${initial_positions}" joint_name_wo_prefix="elbow_joint"/>
-      <xacro:configure_joint joint_name="${tf_prefix}wrist_1_joint"      initial_positions="${initial_positions}" joint_name_wo_prefix="wrist_1_joint"/>
-      <xacro:configure_joint joint_name="${tf_prefix}wrist_2_joint"      initial_positions="${initial_positions}" joint_name_wo_prefix="wrist_2_joint"/>
-      <xacro:configure_joint joint_name="${tf_prefix}wrist_3_joint"      initial_positions="${initial_positions}" joint_name_wo_prefix="wrist_3_joint"/>
+      <xacro:configure_joint joint_name="${tf_prefix}shoulder_pan_joint"
+        initial_positions="${initial_positions}" joint_name_wo_prefix="shoulder_pan_joint" />
+      <xacro:configure_joint joint_name="${tf_prefix}shoulder_lift_joint"
+        initial_positions="${initial_positions}" joint_name_wo_prefix="shoulder_lift_joint" />
+      <xacro:configure_joint joint_name="${tf_prefix}elbow_joint"
+        initial_positions="${initial_positions}" joint_name_wo_prefix="elbow_joint" />
+      <xacro:configure_joint joint_name="${tf_prefix}wrist_1_joint"
+        initial_positions="${initial_positions}" joint_name_wo_prefix="wrist_1_joint" />
+      <xacro:configure_joint joint_name="${tf_prefix}wrist_2_joint"
+        initial_positions="${initial_positions}" joint_name_wo_prefix="wrist_2_joint" />
+      <xacro:configure_joint joint_name="${tf_prefix}wrist_3_joint"
+        initial_positions="${initial_positions}" joint_name_wo_prefix="wrist_3_joint" />
+      <xacro:configure_joint joint_name="${tf_prefix}robotiq_85_left_knuckle_joint"
+        initial_positions="${initial_positions}"
+        joint_name_wo_prefix="robotiq_85_left_knuckle_joint" />
       <sensor name="${tf_prefix}motor_fts">
         <state_interface name="force.x" />

File: models/ur5e/urdf_ros2/ur5e_mujoco.urdf.xacro (robot description, xacro)
@@ -1,5 +1,6 @@
 <?xml version="1.0" encoding='utf-8'?>
 <robot name="ur5e" xmlns:xacro="http://ros.org/wiki/xacro">
-    <xacro:arg name="initial_positions_file" default="$(find mujoco_with_ros2)/config/initial_positions.yaml" />
+    <xacro:arg name="initial_positions_file"
+        default="$(find mujoco_with_ros2)/config/initial_positions.yaml" />
     <xacro:arg name="ros2_control_hardware_type" default="mujoco" />
     <xacro:arg name="tf_prefix" default="" />
@@ -7,11 +8,20 @@
     <!-- Import ur5e urdf file -->
     <xacro:include filename="$(find mujoco_with_ros2)/models/ur5e/urdf_ros2/ur5e_macro.xacro" />
-    <xacro:ur5e name="ur5e" tf_prefix="$(arg tf_prefix)"  connected_to="world"  rpy="0 0 0"  xyz="0 -0.145 0.97"/>
+    <xacro:ur5e name="ur5e" tf_prefix="$(arg tf_prefix)" connected_to="world" rpy="0 0 0"
+        xyz="0 -0.145 0.97" />
     <!-- Import ur5e ros2_control description -->
     <xacro:include filename="$(find mujoco_with_ros2)/models/ur5e/urdf_ros2/ur5e.ros2_control.xacro" />
-    <xacro:include filename="$(find mujoco_with_ros2)/models/ur5e/urdf_ros2/robotiq.ros2_control.xacro" />
-    <xacro:ur5e_ros2_control name="UR5eFakeSystem" initial_positions_file="$(arg initial_positions_file)" ros2_control_hardware_type="$(arg ros2_control_hardware_type)" tf_prefix="$(arg tf_prefix)"/>
-    <!-- <xacro:robotiq_ros2_control name="RobotiqFakeSystem" initial_positions_file="$(arg initial_positions_file)" ros2_control_hardware_type="$(arg ros2_control_hardware_type)" tf_prefix="$(arg tf_prefix)"/> -->
+    <xacro:include
+        filename="$(find mujoco_with_ros2)/models/ur5e/urdf_ros2/robotiq.ros2_control.xacro" />
+    <xacro:ur5e_ros2_control
+        name="UR5eFakeSystem"
+        initial_positions_file="$(arg initial_positions_file)"
+        ros2_control_hardware_type="$(arg ros2_control_hardware_type)"
+        tf_prefix="$(arg tf_prefix)" />
+    <!-- <xacro:robotiq_ros2_control name="RobotiqFakeSystem" initial_positions_file="$(arg
+    initial_positions_file)" ros2_control_hardware_type="$(arg ros2_control_hardware_type)"
+    tf_prefix="$(arg tf_prefix)"/> -->
     <!-- Import d435i/camera file -->
-    <!-- <xacro:include filename="$(find mujoco_with_ros2)/ur_description/urdf/ur5e/d435i_macro.xacro" /> -->
+    <!-- <xacro:include filename="$(find
+    mujoco_with_ros2)/ur_description/urdf/ur5e/d435i_macro.xacro" /> -->
 </robot>
